Commit message: Add collision link for oakd

File: depthai_descriptions/urdf/include/base_macro.urdf.xacro (robot description, xacro)
@@ -37,4 +37,13 @@
                 </material>
             </visual>
+            <collision>
+                <origin
+                    xyz="0 0 0"
+                    rpy="0 0 0" />
+                <geometry>
+                  <mesh
+                      filename="package://rif_gripper_description/meshes/oakd-s2/collision/oakd_link.STL" />
+                </geometry>
+            </collision>
         </link>
         <joint name="${camera_name}_model_origin_joint" type="fixed">
